Commit message: launch 파일 수정

File: src/mobile_manipulator_description/urdf/dofbot.urdf.xacro (robot description, xacro)
@@ -1,10 +1,29 @@
 <?xml version="1.0"?>
 <robot name="dofbot" xmlns:xacro="http://www.ros.org/wiki/xacro">
+    <!-- =================== -->
+    <!-- Property Variables -->
+    <!-- =================== -->
     <xacro:property name="PI" value="3.14159265359"/>
-    <xacro:property name="link_width" value="0.04"/> <link name="manipulator_base_link">
+    <xacro:property name="link_width" value="0.04"/>
+    <xacro:property name="link_length" value="0.2"/>
+    <xacro:property name="base_size" value="0.1"/>
+    <xacro:property name="base_height" value="0.01"/>
+    <!-- =================== -->
+    <!-- Base Link -->
+    <!-- =================== -->
+    <link name="manipulator_base_link">
         <visual>
-            <geometry><box size="0.1 0.1 0.01"/></geometry>
+            <geometry>
+                <box size="${base_size} ${base_size} ${base_height}"/>
+            </geometry>
+            <material name="Gray">
+                <color rgba="0.5 0.5 0.5 1"/>
+            </material>
         </visual>
-        <collision><geometry><box size="0.1 0.1 0.01"/></geometry></collision>
+        <collision>
+            <geometry>
+                <box size="${base_size} ${base_size} ${base_height}"/>
+            </geometry>
+        </collision>
         <inertial>
             <mass value="0.5"/>
@@ -12,14 +31,67 @@
         </inertial>
     </link>
+    <!-- =================== -->
+    <!-- Link1 -->
+    <!-- =================== -->
+    <link name="link1">
+        <visual>
+            <geometry>
+                <box size="${link_width} ${link_width} ${link_length}"/>
+            </geometry>
+            <material name="Blue">
+                <color rgba="0 0 1 1"/>
+            </material>
+        </visual>
+        <collision>
+            <geometry>
+                <box size="${link_width} ${link_width} ${link_length}"/>
+            </geometry>
+        </collision>
+        <inertial>
+            <mass value="0.2"/>
+            <inertia ixx="0.0002" ixy="0" ixz="0" iyy="0.0002" iyz="0" izz="0.0002"/>
+        </inertial>
+    </link>
+    <!-- =================== -->
+    <!-- Link2 -->
+    <!-- =================== -->
+    <link name="link2">
+        <visual>
+            <geometry>
+                <box size="${link_width} ${link_width} ${link_length}"/>
+            </geometry>
+            <material name="Green">
+                <color rgba="0 1 0 1"/>
+            </material>
+        </visual>
+        <collision>
+            <geometry>
+                <box size="${link_width} ${link_width} ${link_length}"/>
+            </geometry>
+        </collision>
+        <inertial>
+            <mass value="0.2"/>
+            <inertia ixx="0.0002" ixy="0" ixz="0" iyy="0.0002" iyz="0" izz="0.0002"/>
+        </inertial>
+    </link>
+    <!-- =================== -->
+    <!-- Joint1: Base -> Link1 -->
+    <!-- =================== -->
     <joint name="joint1" type="revolute">
         <parent link="manipulator_base_link"/>
         <child link="link1"/>
-        <origin xyz="0 0 0.05" rpy="0 0 0"/>
-        <axis xyz="0 0 1"/> <limit lower="-${PI}" upper="${PI}" velocity="0.5" effort="10.0"/>
+        <origin xyz="0 0 ${base_height}" rpy="0 0 0"/>
+        <axis xyz="0 0 1"/>
+        <limit lower="-${PI}" upper="${PI}" velocity="0.5" effort="10.0"/>
     </joint>
+    <!-- =================== -->
+    <!-- Joint2: Link1 -> Link2 -->
+    <!-- =================== -->
     <joint name="joint2" type="revolute">
         <parent link="link1"/>
         <child link="link2"/>
-        <origin xyz="0 0 0.1" rpy="0 0 0"/>
-        <axis xyz="0 1 0"/> <limit lower="-1.57" upper="1.57" velocity="0.5" effort="10.0"/> </joint>
-    </robot>
+        <origin xyz="0 0 ${link_length}" rpy="0 0 0"/>
+        <axis xyz="0 1 0"/>
+        <limit lower="-1.57" upper="1.57" velocity="0.5" effort="10.0"/>
+    </joint>
+</robot>

File: src/mobile_manipulator_description/urdf/mobile_manipulator.urdf.xacro (robot description, xacro)
@@ -2,5 +2,5 @@
 <robot name="mobile_manipulator" xmlns:xacro="http://www.ros.org/wiki/xacro">
     <xacro:property name="PI" value="3.14159265359"/>
-    <xacro:include filename="$(find turtlebot3_description)/urdf/turtlebot3_waffle.urdf.xacro"/>
+    <xacro:include filename="$(find turtlebot3_description)/urdf/turtlebot3_waffle_pi.urdf"/>
     <xacro:include filename="$(find mobile_manipulator_description)/urdf/dofbot.urdf.xacro"/>
     <joint name="manipulator_base_joint" type="fixed">
