Commit message: import 추가

File: src/mobile_manipulator_description/ros2_control/mobile_manipulator.ros2_control.xacro (robot description, xacro)
@@ -1,9 +1,16 @@
 <?xml version="1.0"?>
 <robot name="mobile_manipulator" xmlns:xacro="http://www.ros.org/wiki/xacro">
+    <!-- ========================================================= -->
+    <!--  ROS2 Control System (Mobile Base + DOFbot Arm)          -->
+    <!-- ========================================================= -->
     <xacro:macro name="mobile_manipulator_ros2_control" params="name">
         <ros2_control name="${name}" type="system">
+            <!-- Gazebo ros2_control plugin -->
             <hardware>
                 <plugin>gazebo_ros2_control/GazeboSystem</plugin>
             </hardware>
+            <!-- ========================= -->
+            <!-- 1. TB3 Base Wheel Joints -->
+            <!-- ========================= -->
             <joint name="wheel_left_joint">
                 <command_interface name="velocity">
@@ -22,4 +29,7 @@
                 <state_interface name="position"/>
             </joint>
+            <!-- ========================= -->
+            <!-- 2. DOFbot Manipulator     -->
+            <!-- ========================= -->
             <joint name="joint1">
                 <command_interface name="position">
@@ -30,6 +40,15 @@
                 <state_interface name="velocity"/>
             </joint>
-            </ros2_control>
+            <joint name="joint2">
+                <command_interface name="position">
+                    <param name="min">-1.57</param>
+                    <param name="max">1.57</param>
+                </command_interface>
+                <state_interface name="position"/>
+                <state_interface name="velocity"/>
+            </joint>
+        </ros2_control>
     </xacro:macro>
+    <!-- Macro 실행 -->
     <xacro:mobile_manipulator_ros2_control name="MobileManipulator"/>
 </robot>
